Commit message: add upper arm and isaac sim control with moveit

File: gr1_t2_upper_moveit_config/config/GR1_T2.ros2_control.xacro (robot description, xacro)
@@ -182,4 +182,88 @@
                 <state_interface name="velocity"/>
             </joint>
+            <joint name="l_shoulder_pitch">
+                <command_interface name="position"/>
+                <state_interface name="position">
+                  <param name="initial_value">${initial_positions['l_shoulder_pitch']}</param>
+                </state_interface>
+                <state_interface name="velocity"/>
+            </joint>
+            <joint name="l_shoulder_roll">
+                <command_interface name="position"/>
+                <state_interface name="position">
+                  <param name="initial_value">${initial_positions['l_shoulder_roll']}</param>
+                </state_interface>
+                <state_interface name="velocity"/>
+            </joint>
+            <joint name="l_shoulder_yaw">
+                <command_interface name="position"/>
+                <state_interface name="position">
+                  <param name="initial_value">${initial_positions['l_shoulder_yaw']}</param>
+                </state_interface>
+                <state_interface name="velocity"/>
+            </joint>
+            <joint name="l_elbow_pitch">
+                <command_interface name="position"/>
+                <state_interface name="position">
+                  <param name="initial_value">${initial_positions['l_elbow_pitch']}</param>
+                </state_interface>
+                <state_interface name="velocity"/>
+            </joint>
+            <joint name="l_wrist_yaw">
+                <command_interface name="position"/>
+                <state_interface name="position">
+                  <param name="initial_value">${initial_positions['l_wrist_yaw']}</param>
+                </state_interface>
+                <state_interface name="velocity"/>
+            </joint>
+            <joint name="l_wrist_roll">
+                <command_interface name="position"/>
+                <state_interface name="position">
+                  <param name="initial_value">${initial_positions['l_wrist_roll']}</param>
+                </state_interface>
+                <state_interface name="velocity"/>
+            </joint>
+            <joint name="r_shoulder_pitch">
+                <command_interface name="position"/>
+                <state_interface name="position">
+                  <param name="initial_value">${initial_positions['r_shoulder_pitch']}</param>
+                </state_interface>
+                <state_interface name="velocity"/>
+            </joint>
+            <joint name="r_shoulder_roll">
+                <command_interface name="position"/>
+                <state_interface name="position">
+                  <param name="initial_value">${initial_positions['r_shoulder_roll']}</param>
+                </state_interface>
+                <state_interface name="velocity"/>
+            </joint>
+            <joint name="r_shoulder_yaw">
+                <command_interface name="position"/>
+                <state_interface name="position">
+                  <param name="initial_value">${initial_positions['r_shoulder_yaw']}</param>
+                </state_interface>
+                <state_interface name="velocity"/>
+            </joint>
+            <joint name="r_elbow_pitch">
+                <command_interface name="position"/>
+                <state_interface name="position">
+                  <param name="initial_value">${initial_positions['r_elbow_pitch']}</param>
+                </state_interface>
+                <state_interface name="velocity"/>
+            </joint>
+            <joint name="r_wrist_yaw">
+                <command_interface name="position"/>
+                <state_interface name="position">
+                  <param name="initial_value">${initial_positions['r_wrist_yaw']}</param>
+                </state_interface>
+                <state_interface name="velocity"/>
+            </joint>
+            <joint name="r_wrist_roll">
+                <command_interface name="position"/>
+                <state_interface name="position">
+                  <param name="initial_value">${initial_positions['r_wrist_roll']}</param>
+                </state_interface>
+                <state_interface name="velocity"/>
+            </joint>
         </ros2_control>
     </xacro:macro>

File: humanoid_description/urdf/GR1_T2.ros2_control.xacro (robot description, xacro)
@@ -1,12 +1,16 @@
 <?xml version="1.0"?>
 <robot xmlns:xacro="http://www.ros.org/wiki/xacro">
-  <xacro:macro name="GR1_T2_ros2_control" params="name">
+  <xacro:macro name="GR1_T2_ros2_control" params="name ros2_control_hardware_type">
     <ros2_control name="${name}" type="system">
-      <!-- <hardware>
-        <plugin>dynamixel_hardware/DynamixelHardware</plugin>
-        <param name="usb_port">/dev/ttyUSB0</param>
-        <param name="baud_rate">115200</param>
-        <param name="use_dummy">true</param>
-      </hardware> -->
+      <hardware>
+          <xacro:if value="${ros2_control_hardware_type == 'mock_components'}">
+              <plugin>mock_components/GenericSystem</plugin>
+          </xacro:if>
+          <xacro:if value="${ros2_control_hardware_type == 'isaac'}">
+              <plugin>topic_based_ros2_control/TopicBasedSystem</plugin>
+              <param name="joint_commands_topic">/isaac_joint_commands</param>
+              <param name="joint_states_topic">/isaac_joint_states</param>
+          </xacro:if>
+      </hardware>
       <joint name="L_index_intermediate_joint">
         <command_interface name="position"/>

File: humanoid_description/urdf/GR1_T2.urdf.xacro (robot description, xacro)
@@ -1,4 +1,5 @@
 <?xml version="1.0"?>
 <robot name="GR1_T2" xmlns:xacro="http://ros.org/wiki/xacro">
+  <xacro:arg name="ros2_control_hardware_type" default="mock_components" />
   <xacro:include filename="$(find humanoid_description)/urdf/GR1_T2.xacro" />
   <xacro:include filename="$(find humanoid_description)/urdf/GR1_T2.ros2_control.xacro" />
@@ -7,4 +8,4 @@
     <origin xyz="0 0 0" rpy="0 0 0" />
   </xacro:GR1_T2>
-  <xacro:GR1_T2_ros2_control name="GR1_T2_ros2_control" />
+  <xacro:GR1_T2_ros2_control name="GR1_T2_ros2_control" ros2_control_hardware_type="$(arg ros2_control_hardware_type)" />
 </robot>

Commit message: modify upper moveit config

File: gr1_t2_upper_moveit_config/config/GR1_T2.ros2_control.xacro (robot description, xacro)
@@ -266,4 +266,11 @@
                 <state_interface name="velocity"/>
             </joint>
+            <joint name="r_wrist_pitch">
+                <command_interface name="position"/>
+                <state_interface name="position">
+                  <param name="initial_value">${initial_positions['r_wrist_roll']}</param>
+                </state_interface>
+                <state_interface name="velocity"/>
+            </joint>
         </ros2_control>
     </xacro:macro>

File: humanoid_description/urdf/GR1_T2.ros2_control.xacro (robot description, xacro)
@@ -188,4 +188,11 @@
         <state_interface name="effort"/>
       </joint>
+      <joint name="joint_head_roll">
+        <command_interface name="position"/>
+        <command_interface name="velocity"/>
+        <state_interface name="position"/>
+        <state_interface name="velocity"/>
+        <state_interface name="effort"/>
+      </joint>
       <joint name="joint_waist_pitch">
         <command_interface name="position"/>
@@ -371,4 +378,11 @@
       </joint>
       <joint name="r_wrist_yaw">
+        <command_interface name="position"/>
+        <command_interface name="velocity"/>
+        <state_interface name="position"/>
+        <state_interface name="velocity"/>
+        <state_interface name="effort"/>
+      </joint>
+      <joint name="r_wrist_pitch">
         <command_interface name="position"/>
         <command_interface name="velocity"/>
